File: hardware/power.kicad_sch (KiCad schematic)
At the start: 37 parts, among them J3 Screw_Terminal_01x04, U3 XC6206PxxxMR, U4 AMS1117-5.0, U5 SPX3819M5-L, U7 SPX3819M5-L, U8 INA3221

Commit message: Fix BOM errors
Parts:
- C12, C9: LCSC C1591 -> C59461; MPN CL10B104KB8NNNC -> CL10A226MQ8NRNC
Changed lines of the file:
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@@
       (effects (font (size 1.27 1.27)) hide)
     )
-    (property "MPN" "CL10B104KB8NNNC" (at 137.16 76.2 0)
+    (property "MPN" "CL10A226MQ8NRNC" (at 137.16 76.2 0)
       (effects (font (size 1.27 1.27)) hide)
     )
-    (property "LCSC" "C1591" (at 137.16 76.2 0)
+    (property "LCSC" "C59461" (at 137.16 76.2 0)
       (effects (font (size 1.27 1.27)) hide)
     )
@@
       (effects (font (size 1.27 1.27)) hide)
     )
-    (property "MPN" "CL10B104KB8NNNC" (at 110.49 76.2 0)
+    (property "MPN" "CL10A226MQ8NRNC" (at 110.49 76.2 0)
       (effects (font (size 1.27 1.27)) hide)
     )
-    (property "LCSC" "C1591" (at 110.49 76.2 0)
+    (property "LCSC" "C59461" (at 110.49 76.2 0)
       (effects (font (size 1.27 1.27)) hide)
     )
