File: hardware/power.kicad_sch (KiCad schematic)
At the start: 37 parts, among them J3 Screw_Terminal_01x04, U3 XC6206PxxxMR, U4 AMS1117-5.0, U5 SPX3819M5-L, U7 SPX3819M5-L, U8 INA3221

Commit message: FEM v3 Updates
Other:
- note added: "700mA min for 5VA Amplifiers, attenuator, log detector 0.2 Ohm sense @ 0.6A => 0.12 V Drop (72 mW)"
- note removed: "550mA min for 5VA Amplifiers, attenuator, log detector 0.2 Ohm sense @ 0.6A => 0.12 V Drop (72 mW)"

Commit message: Update FEM hardware design for production version
Parts:
- renumbered C14 to C10, C15 to C11, C2 to C3, C7 to C4, C8 to C5, C9 to C6, C10 to C7, C12 to C8, C13 to C9, H4 to H1, H5 to H2, H6 to H3, H1 to H4, H2 to H5, H3 to H6, J3 to J2, R4 to R3, R5 to R4, R6 to R5, R7 to R6, R16 to R7, U3 to U2, U4 to U3, U5 to U4, U7 to U5, U8 to U6
