File: hardware/lo_filter.kicad_sch (KiCad schematic)
At the start: 5 parts

Commit message: Update FEM hardware design for production version
Parts:
- renumbered C89 to C63, C90 to C64, C91 to C65, L27 to L26, L28 to L27
Changed lines of the file:
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@@
   (symbol (lib_id "power:GND") (at 113.03 104.14 0) (unit 1)
     (in_bom yes) (on_board yes) (dnp no) (fields_autoplaced)
-    (property "Reference" "#PWR0186" (at 113.03 110.49 0)
+    (property "Reference" "#PWR099" (at 113.03 110.49 0)
       (effects (font (size 1.27 1.27)) hide)
     )
@@
       (project "GreX Frontend"
         (path "/e63e39d7-6ac0-4ffd-8aa3-1841a4541b55/546148dc-8a5c-4178-ace4-1d6889891417/63a821c0-1ea4-41d0-8e0f-5a0b95760f51"
-          (reference "#PWR0186") (unit 1)
+          (reference "#PWR099") (unit 1)
         )
       )
@@
   (symbol (lib_id "power:GND") (at 130.81 104.14 0) (unit 1)
     (in_bom yes) (on_board yes) (dnp no) (fields_autoplaced)
-    (property "Reference" "#PWR0187" (at 130.81 110.49 0)
+    (property "Reference" "#PWR0100" (at 130.81 110.49 0)
       (effects (font (size 1.27 1.27)) hide)
     )
@@
       (project "GreX Frontend"
         (path "/e63e39d7-6ac0-4ffd-8aa3-1841a4541b55/546148dc-8a5c-4178-ace4-1d6889891417/63a821c0-1ea4-41d0-8e0f-5a0b95760f51"
-          (reference "#PWR0187") (unit 1)
+          (reference "#PWR0100") (unit 1)
         )
       )
@@
   (symbol (lib_id "Device:L") (at 139.7 95.25 90) (unit 1)
     (in_bom yes) (on_board yes) (dnp no) (fields_autoplaced)
-    (property "Reference" "L28" (at 139.7 88.9 90)
+    (property "Reference" "L27" (at 139.7 88.9 90)
       (effects (font (size 1.27 1.27)))
     )
@@
       (project "GreX Frontend"
         (path "/e63e39d7-6ac0-4ffd-8aa3-1841a4541b55/546148dc-8a5c-4178-ace4-1d6889891417/63a821c0-1ea4-41d0-8e0f-5a0b95760f51"
-          (reference "L28") (unit 1)
+          (reference "L27") (unit 1)
         )
       )
@@
   (symbol (lib_id "Device:C") (at 113.03 99.06 0) (unit 1)
     (in_bom yes) (on_board yes) (dnp no) (fields_autoplaced)
-    (property "Reference" "C89" (at 116.84 97.7899 0)
+    (property "Reference" "C63" (at 116.84 97.7899 0)
       (effects (font (size 1.27 1.27)) (justify left))
     )
@@
       (project "GreX Frontend"
         (path "/e63e39d7-6ac0-4ffd-8aa3-1841a4541b55/546148dc-8a5c-4178-ace4-1d6889891417/63a821c0-1ea4-41d0-8e0f-5a0b95760f51"
-          (reference "C89") (unit 1)
+          (reference "C63") (unit 1)
         )
       )
@@
   (symbol (lib_id "Device:C") (at 130.81 99.06 0) (unit 1)
     (in_bom yes) (on_board yes) (dnp no) (fields_autoplaced)
-    (property "Reference" "C90" (at 134.62 97.7899 0)
+    (property "Reference" "C64" (at 134.62 97.7899 0)
       (effects (font (size 1.27 1.27)) (justify left))
     )
@@
       (project "GreX Frontend"
         (path "/e63e39d7-6ac0-4ffd-8aa3-1841a4541b55/546148dc-8a5c-4178-ace4-1d6889891417/63a821c0-1ea4-41d0-8e0f-5a0b95760f51"
-          (reference "C90") (unit 1)
+          (reference "C64") (unit 1)
         )
       )
@@
   (symbol (lib_id "power:GND") (at 147.32 104.14 0) (unit 1)
     (in_bom yes) (on_board yes) (dnp no) (fields_autoplaced)
-    (property "Reference" "#PWR0188" (at 147.32 110.49 0)
+    (property "Reference" "#PWR0101" (at 147.32 110.49 0)
       (effects (font (size 1.27 1.27)) hide)
     )
@@
       (project "GreX Frontend"
         (path "/e63e39d7-6ac0-4ffd-8aa3-1841a4541b55/546148dc-8a5c-4178-ace4-1d6889891417/63a821c0-1ea4-41d0-8e0f-5a0b95760f51"
-          (reference "#PWR0188") (unit 1)
+          (reference "#PWR0101") (unit 1)
         )
       )
@@
   (symbol (lib_id "Device:L") (at 121.92 95.25 90) (unit 1)
     (in_bom yes) (on_board yes) (dnp no) (fields_autoplaced)
-    (property "Reference" "L27" (at 121.92 88.9 90)
+    (property "Reference" "L26" (at 121.92 88.9 90)
       (effects (font (size 1.27 1.27)))
     )
@@
       (project "GreX Frontend"
         (path "/e63e39d7-6ac0-4ffd-8aa3-1841a4541b55/546148dc-8a5c-4178-ace4-1d6889891417/63a821c0-1ea4-41d0-8e0f-5a0b95760f51"
-          (reference "L27") (unit 1)
+          (reference "L26") (unit 1)
         )
       )
@@
   (symbol (lib_id "Device:C") (at 147.32 99.06 0) (unit 1)
     (in_bom yes) (on_board yes) (dnp no) (fields_autoplaced)
-    (property "Reference" "C91" (at 151.13 97.7899 0)
+    (property "Reference" "C65" (at 151.13 97.7899 0)
       (effects (font (size 1.27 1.27)) (justify left))
     )
@@
       (project "GreX Frontend"
         (path "/e63e39d7-6ac0-4ffd-8aa3-1841a4541b55/546148dc-8a5c-4178-ace4-1d6889891417/63a821c0-1ea4-41d0-8e0f-5a0b95760f51"
-          (reference "C91") (unit 1)
-        )
-      )
+          (reference "C65") (unit 1)
+        )
+      )
