File: hardware/power_sense.kicad_sch (KiCad schematic)
At the start: 5 parts, among them U27 AD8314

Commit message: FEM v3 Updates
Parts:
- R38: value 28.7 -> 28

Commit message: Update FEM hardware design for production version
Parts:
- renumbered C99 to C87, C100 to C88, R36 to R25, R38 to R26, U27 to U26
Changed lines of the file:
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@@
   (symbol (lib_id "Device:C") (at 148.59 106.68 90) (unit 1)
     (in_bom yes) (on_board yes) (dnp no)
-    (property "Reference" "C100" (at 151.13 107.95 90)
+    (property "Reference" "C88" (at 151.13 107.95 90)
       (effects (font (size 1.27 1.27)))
     )
@@
       (project "GreX Frontend"
         (path "/e63e39d7-6ac0-4ffd-8aa3-1841a4541b55/546148dc-8a5c-4178-ace4-1d6889891417/eaccd376-6e64-4454-b62f-a0a0f7d65f22/199b51ab-5177-4451-b53f-6e0b743cb47d"
-          (reference "C100") (unit 1)
-        )
-        (path "/e63e39d7-6ac0-4ffd-8aa3-1841a4541b55/546148dc-8a5c-4178-ace4-1d6889891417/73736f53-e594-47a6-b1b8-fbf51934708f/199b51ab-5177-4451-b53f-6e0b743cb47d"
           (reference "C88") (unit 1)
         )
+        (path "/e63e39d7-6ac0-4ffd-8aa3-1841a4541b55/546148dc-8a5c-4178-ace4-1d6889891417/73736f53-e594-47a6-b1b8-fbf51934708f/199b51ab-5177-4451-b53f-6e0b743cb47d"
+          (reference "C83") (unit 1)
+        )
       )
     )
@@
   (symbol (lib_id "Device:C") (at 113.03 106.68 180) (unit 1)
     (in_bom yes) (on_board yes) (dnp no)
-    (property "Reference" "C99" (at 106.68 104.775 0)
+    (property "Reference" "C87" (at 106.68 104.775 0)
       (effects (font (size 1.27 1.27)) (justify right))
     )
@@
       (project "GreX Frontend"
         (path "/e63e39d7-6ac0-4ffd-8aa3-1841a4541b55/546148dc-8a5c-4178-ace4-1d6889891417/eaccd376-6e64-4454-b62f-a0a0f7d65f22/199b51ab-5177-4451-b53f-6e0b743cb47d"
-          (reference "C99") (unit 1)
-        )
-        (path "/e63e39d7-6ac0-4ffd-8aa3-1841a4541b55/546148dc-8a5c-4178-ace4-1d6889891417/73736f53-e594-47a6-b1b8-fbf51934708f/199b51ab-5177-4451-b53f-6e0b743cb47d"
-          (reference "C85") (unit 1)
+          (reference "C87") (unit 1)
+        )
+        (path "/e63e39d7-6ac0-4ffd-8aa3-1841a4541b55/546148dc-8a5c-4178-ace4-1d6889891417/73736f53-e594-47a6-b1b8-fbf51934708f/199b51ab-5177-4451-b53f-6e0b743cb47d"
+          (reference "C82") (unit 1)
         )
       )
@@
   (symbol (lib_id "power:GND") (at 158.75 110.49 0) (unit 1)
     (in_bom yes) (on_board yes) (dnp no) (fields_autoplaced)
-    (property "Reference" "#PWR0206" (at 158.75 116.84 0)
+    (property "Reference" "#PWR0137" (at 158.75 116.84 0)
       (effects (font (size 1.27 1.27)) hide)
     )
@@
       (project "GreX Frontend"
         (path "/e63e39d7-6ac0-4ffd-8aa3-1841a4541b55/546148dc-8a5c-4178-ace4-1d6889891417/eaccd376-6e64-4454-b62f-a0a0f7d65f22/199b51ab-5177-4451-b53f-6e0b743cb47d"
-          (reference "#PWR0206") (unit 1)
-        )
-        (path "/e63e39d7-6ac0-4ffd-8aa3-1841a4541b55/546148dc-8a5c-4178-ace4-1d6889891417/73736f53-e594-47a6-b1b8-fbf51934708f/199b51ab-5177-4451-b53f-6e0b743cb47d"
-          (reference "#PWR0202") (unit 1)
+          (reference "#PWR0137") (unit 1)
+        )
+        (path "/e63e39d7-6ac0-4ffd-8aa3-1841a4541b55/546148dc-8a5c-4178-ace4-1d6889891417/73736f53-e594-47a6-b1b8-fbf51934708f/199b51ab-5177-4451-b53f-6e0b743cb47d"
+          (reference "#PWR0127") (unit 1)
         )
       )
@@
   (symbol (lib_id "power:+5VA") (at 120.65 93.98 0) (unit 1)
     (in_bom yes) (on_board yes) (dnp no)
-    (property "Reference" "#PWR0205" (at 120.65 97.79 0)
+    (property "Reference" "#PWR0135" (at 120.65 97.79 0)
       (effects (font (size 1.27 1.27)) hide)
     )
@@
       (project "GreX Frontend"
         (path "/e63e39d7-6ac0-4ffd-8aa3-1841a4541b55/546148dc-8a5c-4178-ace4-1d6889891417/eaccd376-6e64-4454-b62f-a0a0f7d65f22/199b51ab-5177-4451-b53f-6e0b743cb47d"
-          (reference "#PWR0205") (unit 1)
-        )
-        (path "/e63e39d7-6ac0-4ffd-8aa3-1841a4541b55/546148dc-8a5c-4178-ace4-1d6889891417/73736f53-e594-47a6-b1b8-fbf51934708f/199b51ab-5177-4451-b53f-6e0b743cb47d"
-          (reference "#PWR0190") (unit 1)
+          (reference "#PWR0135") (unit 1)
+        )
+        (path "/e63e39d7-6ac0-4ffd-8aa3-1841a4541b55/546148dc-8a5c-4178-ace4-1d6889891417/73736f53-e594-47a6-b1b8-fbf51934708f/199b51ab-5177-4451-b53f-6e0b743cb47d"
+          (reference "#PWR0125") (unit 1)
         )
       )
@@
   (symbol (lib_id "Project Library:AD8314") (at 134.62 102.87 0) (mirror y) (unit 1)
     (in_bom yes) (on_board yes) (dnp no) (fields_autoplaced)
-    (property "Reference" "U27" (at 133.985 91.44 0)
+    (property "Reference" "U26" (at 133.985 91.44 0)
       (effects (font (size 1.27 1.27)))
     )
@@
       (project "GreX Frontend"
         (path "/e63e39d7-6ac0-4ffd-8aa3-1841a4541b55/546148dc-8a5c-4178-ace4-1d6889891417/eaccd376-6e64-4454-b62f-a0a0f7d65f22/199b51ab-5177-4451-b53f-6e0b743cb47d"
-          (reference "U27") (unit 1)
+          (reference "U26") (unit 1)
         )
         (path "/e63e39d7-6ac0-4ffd-8aa3-1841a4541b55/546148dc-8a5c-4178-ace4-1d6889891417/73736f53-e594-47a6-b1b8-fbf51934708f/199b51ab-5177-4451-b53f-6e0b743cb47d"
@@
   (symbol (lib_id "Device:R") (at 158.75 83.82 0) (unit 1)
     (in_bom yes) (on_board yes) (dnp no) (fields_autoplaced)
-    (property "Reference" "R36" (at 161.29 82.5499 0)
+    (property "Reference" "R25" (at 161.29 82.5499 0)
       (effects (font (size 1.27 1.27)) (justify left))
     )
@@
       (project "GreX Frontend"
         (path "/e63e39d7-6ac0-4ffd-8aa3-1841a4541b55/546148dc-8a5c-4178-ace4-1d6889891417/eaccd376-6e64-4454-b62f-a0a0f7d65f22/199b51ab-5177-4451-b53f-6e0b743cb47d"
-          (reference "R36") (unit 1)
-        )
-        (path "/e63e39d7-6ac0-4ffd-8aa3-1841a4541b55/546148dc-8a5c-4178-ace4-1d6889891417/73736f53-e594-47a6-b1b8-fbf51934708f/199b51ab-5177-4451-b53f-6e0b743cb47d"
-          (reference "R3") (unit 1)
+          (reference "R25") (unit 1)
+        )
+        (path "/e63e39d7-6ac0-4ffd-8aa3-1841a4541b55/546148dc-8a5c-4178-ace4-1d6889891417/73736f53-e594-47a6-b1b8-fbf51934708f/199b51ab-5177-4451-b53f-6e0b743cb47d"
+          (reference "R23") (unit 1)
         )
       )
@@
   (symbol (lib_id "Device:R") (at 158.75 105.41 180) (unit 1)
     (in_bom yes) (on_board yes) (dnp no) (fields_autoplaced)
-    (property "Reference" "R38" (at 161.29 104.775 0)
+    (property "Reference" "R26" (at 161.29 104.775 0)
       (effects (font (size 1.27 1.27)) (justify right))
     )
@@
       (project "GreX Frontend"
         (path "/e63e39d7-6ac0-4ffd-8aa3-1841a4541b55/546148dc-8a5c-4178-ace4-1d6889891417/eaccd376-6e64-4454-b62f-a0a0f7d65f22/199b51ab-5177-4451-b53f-6e0b743cb47d"
-          (reference "R38") (unit 1)
-        )
-        (path "/e63e39d7-6ac0-4ffd-8aa3-1841a4541b55/546148dc-8a5c-4178-ace4-1d6889891417/73736f53-e594-47a6-b1b8-fbf51934708f/199b51ab-5177-4451-b53f-6e0b743cb47d"
-          (reference "R18") (unit 1)
+          (reference "R26") (unit 1)
+        )
+        (path "/e63e39d7-6ac0-4ffd-8aa3-1841a4541b55/546148dc-8a5c-4178-ace4-1d6889891417/73736f53-e594-47a6-b1b8-fbf51934708f/199b51ab-5177-4451-b53f-6e0b743cb47d"
+          (reference "R24") (unit 1)
         )
       )
@@
   (symbol (lib_id "power:GND") (at 113.03 110.49 0) (unit 1)
     (in_bom yes) (on_board yes) (dnp no)
-    (property "Reference" "#PWR0207" (at 113.03 116.84 0)
+    (property "Reference" "#PWR0134" (at 113.03 116.84 0)
       (effects (font (size 1.27 1.27)) hide)
     )
@@
       (project "GreX Frontend"
         (path "/e63e39d7-6ac0-4ffd-8aa3-1841a4541b55/546148dc-8a5c-4178-ace4-1d6889891417/eaccd376-6e64-4454-b62f-a0a0f7d65f22/199b51ab-5177-4451-b53f-6e0b743cb47d"
-          (reference "#PWR0207") (unit 1)
-        )
-        (path "/e63e39d7-6ac0-4ffd-8aa3-1841a4541b55/546148dc-8a5c-4178-ace4-1d6889891417/73736f53-e594-47a6-b1b8-fbf51934708f/199b51ab-5177-4451-b53f-6e0b743cb47d"
-          (reference "#PWR0203") (unit 1)
+          (reference "#PWR0134") (unit 1)
+        )
+        (path "/e63e39d7-6ac0-4ffd-8aa3-1841a4541b55/546148dc-8a5c-4178-ace4-1d6889891417/73736f53-e594-47a6-b1b8-fbf51934708f/199b51ab-5177-4451-b53f-6e0b743cb47d"
+          (reference "#PWR0124") (unit 1)
         )
       )
@@
   (symbol (lib_id "power:GND") (at 123.19 121.92 0) (unit 1)
     (in_bom yes) (on_board yes) (dnp no)
-    (property "Reference" "#PWR0208" (at 123.19 128.27 0)
+    (property "Reference" "#PWR0136" (at 123.19 128.27 0)
       (effects (font (size 1.27 1.27)) hide)
     )
@@
       (project "GreX Frontend"
         (path "/e63e39d7-6ac0-4ffd-8aa3-1841a4541b55/546148dc-8a5c-4178-ace4-1d6889891417/eaccd376-6e64-4454-b62f-a0a0f7d65f22/199b51ab-5177-4451-b53f-6e0b743cb47d"
-          (reference "#PWR0208") (unit 1)
-        )
-        (path "/e63e39d7-6ac0-4ffd-8aa3-1841a4541b55/546148dc-8a5c-4178-ace4-1d6889891417/73736f53-e594-47a6-b1b8-fbf51934708f/199b51ab-5177-4451-b53f-6e0b743cb47d"
-          (reference "#PWR0204") (unit 1)
-        )
-      )
+          (reference "#PWR0136") (unit 1)
+        )
+        (path "/e63e39d7-6ac0-4ffd-8aa3-1841a4541b55/546148dc-8a5c-4178-ace4-1d6889891417/73736f53-e594-47a6-b1b8-fbf51934708f/199b51ab-5177-4451-b53f-6e0b743cb47d"
+          (reference "#PWR0126") (unit 1)
+        )
+      )
